File: Project 3 MCUdatalogger/Project 3 MCUdatalogger.kicad_sch (KiCad schematic)
At the start: 25 parts, among them U1 24LC1025, U2 DS1337S_, U3 24LC1025, U4 ATMEGA328P-AU, Y1 32.768 KHz, Y2 16 MHz

Commit message: Completed Comments
Other:
- note added: "EEPROM"
- note added: "MCU"
- note added: "Mounting"
- note added: "Real Time Clock"
- moved on the sheet: C1, H1, H2, H3, H4, R1, R2, U2, Y1
