File: Project 3 MCUdatalogger/Project 3 MCUdatalogger.kicad_sch (KiCad schematic)
At the start: 25 parts, among them U1 24LC1025, U2 DS1337S_, U3 24LC1025, U4 ATMEGA328P-AU, Y1 32.768 KHz, Y2 16 MHz

Commit message: Routing
Changed lines of the file:
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@@
+	)
+	(junction
+		(at 234.95 38.735)
+		(diameter 0)
+		(color 0 0 0 0)
 	)
 	(junction
@@
 	(wire
 		(pts
+			(xy 234.95 38.735) (xy 234.95 57.15)
+		)
+		(stroke
+			(width 0)
+			(type default)
+		)
+	)
+	(wire
+		(pts
 			(xy 219.075 84.455) (xy 222.25 84.455)
 		)
@@
 	(wire
 		(pts
-			(xy 222.25 38.1) (xy 234.95 38.1)
+			(xy 222.25 38.735) (xy 234.95 38.735)
 		)
 		(stroke
@@
 	(wire
 		(pts
-			(xy 222.25 38.1) (xy 222.25 38.735)
-		)
-		(stroke
-			(width 0)
-			(type default)
-		)
-	)
-	(wire
-		(pts
 			(xy 81.915 63.5) (xy 81.915 62.865)
 		)
@@
 	(wire
 		(pts
-			(xy 234.95 38.1) (xy 234.95 57.15)
-		)
-		(stroke
+			(xy 234.95 38.1) (xy 234.95 38.735)
+		)
+		(stroke
